File: Hardware/Eagle/simple_eq_5532.brd (EAGLE design)
At the start: 100 x 19.1 mm, 43 parts, among them IC1 NE5532, IC2 NE5532

Commit message: Rev 1.1 updated Thonkiconn socket outlines
Parts:
- BAX_IN, BAX_OUT, TILT_IN, TILT_OUT: value (none) -> WQP-PJ301M-12_JACK; device TomW:THONKICONN -> thonkiconn:WQP-PJ301M-12_JACK
Connections:
- net BAX$1: now also BAX_IN.P$1; no longer BAX_IN.P$3
- net BAX$2: now also BAX_OUT.P$1; no longer BAX_OUT.P$3
- net GND: now also BAX_IN.P$3, BAX_OUT.P$3, TILT_IN.P$3, TILT_OUT.P$3; no longer BAX_IN.P$1, BAX_OUT.P$1, TILT_IN.P$1, TILT_OUT.P$1
- net N$5: now also TILT_OUT.P$1; no longer TILT_OUT.P$3
- net N$6: now also TILT_IN.P$1; no longer TILT_IN.P$3
Other:
- board text added: "Simple EQ Designed in Herne Hill, London By Tom Whitwell, March 2014 musicthing.co.uk PCB Rev 1.1"
- board text removed: "Simple EQ Designed in Herne Hill, London By Tom Whitwell, March 2014 musicthing.co.uk"
Changed lines of the file:
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@@
 <?xml version="1.0" encoding="utf-8"?>
 <!DOCTYPE eagle SYSTEM "eagle.dtd">
-<eagle version="6.5.0">
+<eagle version="6.6.0">
 <drawing>
 <settings>
@@
 <layer number="54" name="bGND_GNDA" color="1" fill="9" visible="no" active="no"/>
 <layer number="56" name="wert" color="7" fill="1" visible="no" active="no"/>
+<layer number="57" name="tCAD" color="7" fill="1" visible="no" active="no"/>
 <layer number="91" name="Nets" color="2" fill="1" visible="no" active="no"/>
 <layer number="92" name="Busses" color="1" fill="1" visible="no" active="no"/>
@@
 <layer number="108" name="tplace-old" color="10" fill="1" visible="yes" active="yes"/>
 <layer number="109" name="ref-old" color="11" fill="1" visible="yes" active="yes"/>
+<layer number="110" name="110" color="7" fill="1" visible="no" active="no"/>
+<layer number="111" name="111" color="7" fill="1" visible="no" active="no"/>
+<layer number="112" name="tSilk" color="7" fill="1" visible="no" active="no"/>
 <layer number="116" name="Patch_BOT" color="9" fill="4" visible="yes" active="yes"/>
+<layer number="118" name="Rect_Pads" color="7" fill="1" visible="no" active="no"/>
 <layer number="121" name="_tsilk" color="7" fill="1" visible="yes" active="yes"/>
 <layer number="122" name="_bsilk" color="7" fill="1" visible="yes" active="yes"/>
+<layer number="123" name="tTestmark" color="7" fill="1" visible="no" active="no"/>
+<layer number="124" name="bTestmark" color="7" fill="1" visible="no" active="no"/>
 <layer number="125" name="_tNames" color="7" fill="1" visible="yes" active="yes"/>
+<layer number="126" name="_bNames" color="7" fill="1" visible="no" active="no"/>
+<layer number="127" name="_tValues" color="7" fill="1" visible="no" active="no"/>
+<layer number="128" name="_bValues" color="7" fill="1" visible="no" active="no"/>
+<layer number="131" name="prix" color="7" fill="1" visible="yes" active="yes"/>
+<layer number="132" name="test" color="7" fill="1" visible="yes" active="yes"/>
 <layer number="144" name="Drill_legend" color="7" fill="1" visible="yes" active="yes"/>
+<layer number="150" name="Notes" color="7" fill="1" visible="yes" active="yes"/>
 <layer number="151" name="HeatSink" color="7" fill="1" visible="yes" active="yes"/>
+<layer number="152" name="_bDocu" color="7" fill="1" visible="no" active="no"/>
+<layer number="153" name="FabDoc1" color="6" fill="1" visible="no" active="no"/>
+<layer number="154" name="FabDoc2" color="2" fill="1" visible="no" active="no"/>
+<layer number="155" name="FabDoc3" color="7" fill="15" visible="no" active="no"/>
 <layer number="199" name="Contour" color="7" fill="1" visible="yes" active="yes"/>
 <layer number="200" name="200bmp" color="1" fill="10" visible="yes" active="yes"/>
@@
 <layer number="223" name="223bmp" color="24" fill="1" visible="no" active="no"/>
 <layer number="224" name="224bmp" color="25" fill="1" visible="no" active="no"/>
+<layer number="248" name="Housing" color="7" fill="1" visible="no" active="no"/>
+<layer number="249" name="Edge" color="7" fill="1" visible="no" active="no"/>
 <layer number="250" name="Descript" color="3" fill="1" visible="no" active="no"/>
 <layer number="251" name="SMDround" color="12" fill="11" visible="no" active="no"/>
@@
 <wire x1="0" y1="19.05" x2="0" y2="0" width="0" layer="20"/>
 <text x="40.6654" y="0.5842" size="0.6096" layer="21">Simple EQ Designed in Herne Hill, London
-By Tom Whitwell, March 2014 musicthing.co.uk</text>
+By Tom Whitwell, March 2014 musicthing.co.uk
+PCB Rev 1.1</text>
 <wire x1="0" y1="9.525" x2="100" y2="9.525" width="0.0254" layer="51"/>
 </plain>
@@
 <element name="R7" library="TomW" package="R0805" value="" x="62.23" y="16.51"/>
 <element name="C4" library="TomW" package="R0805" value="22pf" x="60.96" y="10.16" rot="R270"/>
-<element name="BAX_IN" library="TomW" package="THONKICONN" value="" x="20.32" y="4.572" rot="MR270"/>
+<element name="BAX_IN" library="thonkiconn" package="WQP-PJ301M-12_JACK" value="WQP-PJ301M-12_JACK" x="20.32" y="4.572" rot="MR270"/>
 <element name="R13" library="TomW" package="R0805" value="220R" x="15.875" y="9.525" rot="R270"/>
-<element name="BAX_OUT" library="TomW" package="THONKICONN" value="" x="20.32" y="14.478" rot="MR270"/>
+<element name="BAX_OUT" library="thonkiconn" package="WQP-PJ301M-12_JACK" value="WQP-PJ301M-12_JACK" x="20.32" y="14.478" rot="MR270"/>
 <element name="R2" library="TomW" package="R0805" value="10k" x="4.445" y="1.905"/>
 <element name="R4" library="TomW" package="R0805" value="10k" x="19.05" y="9.525" rot="R270"/>
@@
 <element name="R12" library="TomW" package="R0805" value="6.8k" x="33.274" y="14.732"/>
 <element name="C6" library="TomW" package="R0805" value="22pf" x="34.29" y="10.16" rot="R90"/>
-<element name="TILT_IN" library="TomW" package="THONKICONN" value="" x="6.096" y="4.572" rot="MR270"/>
+<element name="TILT_IN" library="thonkiconn" package="WQP-PJ301M-12_JACK" value="WQP-PJ301M-12_JACK" x="6.096" y="4.572" rot="MR270"/>
 <element name="R14" library="TomW" package="R0805" value="220R" x="3.81" y="11.303" smashed="yes">
 <attribute name="NAME" x="1.51095625" y="10.16390625" size="0.635" layer="25" rot="R90"/>
 <attribute name="VALUE" x="7.489765625" y="10.13118125" size="0.635" layer="27" rot="R90"/>
 </element>
-<element name="TILT_OUT" library="TomW" package="THONKICONN" value="" x="6.096" y="14.478" rot="MR270"/>
+<element name="TILT_OUT" library="thonkiconn" package="WQP-PJ301M-12_JACK" value="WQP-PJ301M-12_JACK" x="6.096" y="14.478" rot="MR270"/>
 <element name="POWER" library="TomW" package="MA05-2" value="" x="83.82" y="16.51" locked="yes">
 <attribute name="OC_NEWARK" value="unknown" x="128.27" y="-15.24" size="1.778" layer="27" display="off"/>
@@
 <contactref element="IC1" pad="3"/>
 <contactref element="IC1" pad="5"/>
-<contactref element="BAX_IN" pad="P$1"/>
-<contactref element="BAX_OUT" pad="P$1"/>
+<contactref element="BAX_IN" pad="P$3"/>
+<contactref element="BAX_OUT" pad="P$3"/>
 <contactref element="IC2" pad="3"/>
 <contactref element="IC2" pad="5"/>
-<contactref element="TILT_OUT" pad="P$1"/>
-<contactref element="TILT_IN" pad="P$1"/>
+<contactref element="TILT_OUT" pad="P$3"/>
+<contactref element="TILT_IN" pad="P$3"/>
 <contactref element="POWER" pad="7"/>
 <contactref element="POWER" pad="5"/>
@@
 <signal name="BAX$1">
 <contactref element="R1" pad="2"/>
-<contactref element="BAX_IN" pad="P$3"/>
+<contactref element="BAX_IN" pad="P$1"/>
 <wire x1="12.7" y1="8.575" x2="12.7" y2="7.637490625" width="0.4064" layer="1"/>
 <wire x1="12.7" y1="7.637490625" x2="12.901871875" y2="7.150128125" width="0.4064" layer="1" curve="44.999816"/>
-<wire x1="12.901871875" y1="7.150128125" x2="15.48" y2="4.572" width="0.4064" layer="1"/>
+<wire x1="12.901871875" y1="7.150128125" x2="15.32" y2="4.572" width="0.4064" layer="1"/>
 </signal>
 <signal name="BAX$2">
 <contactref element="R13" pad="1"/>
-<contactref element="BAX_OUT" pad="P$3"/>
-<wire x1="15.48" y1="14.478" x2="15.48" y2="10.87" width="0.4064" layer="1"/>
+<contactref element="BAX_OUT" pad="P$1"/>
+<wire x1="15.32" y1="14.478" x2="15.48" y2="10.87" width="0.4064" layer="1"/>
 <wire x1="15.48" y1="10.87" x2="15.875" y2="10.475" width="0.4064" layer="1"/>
 </signal>
@@
 <signal name="N$5">
 <contactref element="R14" pad="1"/>
-<contactref element="TILT_OUT" pad="P$3"/>
+<contactref element="TILT_OUT" pad="P$1"/>
 <wire x1="2.86" y1="11.303" x2="2.86" y2="12.4719125" width="0.4064" layer="1"/>
 <wire x1="2.86" y1="12.4719125" x2="2.57568125" y2="13.15831875" width="0.4064" layer="1" curve="45.00013"/>
-<wire x1="2.57568125" y1="13.15831875" x2="1.256" y2="14.478" width="0.4064" layer="1"/>
+<wire x1="2.57568125" y1="13.15831875" x2="1.096" y2="14.478" width="0.4064" layer="1"/>
 </signal>
 <signal name="N$6">
 <contactref element="R2" pad="1"/>
-<contactref element="TILT_IN" pad="P$3"/>
+<contactref element="TILT_IN" pad="P$1"/>
 <wire x1="3.495" y1="1.905" x2="3.495" y2="2.573021875" width="0.4064" layer="1"/>
 <wire x1="3.495" y1="2.573021875" x2="2.375834375" y2="4.167378125" width="0.4064" layer="1" curve="70.134129"/>
-<wire x1="2.375834375" y1="4.167378125" x2="1.256" y2="4.572" width="0.4064" layer="1"/>
+<wire x1="2.375834375" y1="4.167378125" x2="1.096" y2="4.572" width="0.4064" layer="1"/>
 </signal>
 <signal name="+12V" class="3">
